File: Coax Switch Controller/Coax Switch Controller.kicad_sch (KiCad schematic)
At the start: 133 parts, among them J1 8P8C, J2 8P8C, J3 Screw_Terminal_01x02, Q1 MMBT3904, Q10 MMBT3904, Q11 MMBT3904, Q12 MMBT3904, Q13 DMP2004K-7, Q14 DMP2004K-7, Q15 DMP2004K-7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

Commit message: Updated to Kicad 8. Added bill of materials, and PCB's of the output.
Parts:
- C1, C3, C6: DigiKey-PN (none) -> PCE3795CT-ND
- C2, C4, C5, C7, C8, C9: DigiKey-PN (none) -> C0603C103J5REC7411
- D1, D10, D11, D12, D2, D3, D4, D5, D6, D7, D8, D9: value MRA4007T3G -> 1N4007; DigiKey-PN (none) -> 1655-1N4007FLCT-ND
- D13, D14, D15, D16, D17, D18, D19, D20, D21, D22, D23, D24: DigiKey-PN (none) -> 732-4985-1-ND
- D25: DigiKey-PN (none) -> 1655-1N4007FLCT-ND
- FB1, FB10, FB11, FB12, FB13, FB14, FB15, FB16, FB2, FB3, FB4, FB5, FB6, FB7, FB8, FB9: DigiKey-PN (none) -> 240-2411-1-ND
- J1, J2: DigiKey-PN (none) -> 609-1046-ND
- J3: DigiKey-PN (none) -> 732-10955-ND
- Q1, Q10, Q11, Q12, Q2, Q3, Q4, Q5, Q6, Q7, Q8, Q9: DigiKey-PN (none) -> MMBT3904TPMSCT-ND
- Q13, Q14, Q15, Q16, Q17, Q18, Q19, Q20, Q21, Q22, Q23, Q24: DigiKey-PN (none) -> DMP2004KDICT-ND
- R1, R10, R11, R12, R2, R3, R4, R5, R6, R7, R8, R9: DigiKey-PN (none) -> 311-4.70KCRCT-ND
- R13, R14, R15, R16, R17, R18, R19, R20, R21, R22, R23, R24: DigiKey-PN (none) -> 311-100KARCT-ND
- R25, R26, R27, R28, R29, R30, R31, R32, R33, R34, R35, R36: DigiKey-PN (none) -> 311-10.0KCRCT-ND
- R37, R38, R39, R40, R41, R42, R43, R44, R45, R46, R47, R48: DigiKey-PN (none) -> 311-1.00KCRCT-ND
- U1: SparkFun-PN (none) -> SPX-18018
- U2, U3: DigiKey-PN (none) -> 296-9188-5-ND
- U4: DigiKey-PN (none) -> LM1086ISX-5.0/NOPBCT-ND
